File: hardware/di8.kicad_pcb (KiCad board)
At the start: 4 copper layers, 100 x 85 mm, 131 parts, among them J101 TNG-Power-TOP, J102 TNG-Power-BTM, J103 TNG-Data-TOP, J104 TNG-Data-BTM, P102 Debug, P103 PE, P201 INPUT0, P202 INPUT1, P203 INPUT2, P204 INPUT3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

Commit message: fix inductor footprints
Parts:
- LED101: footprint kicad-libraries:LED-RGB-LP -> LED-RGB-LP
- turned T101 to 180 degrees
Connections:
- T101 pad 1: Net-(C120-Pad2) -> Net-(C121-Pad1)
- T101 pad 3: Net-(C121-Pad1) -> Net-(C120-Pad2)
Changed lines of the file:
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@@
   (page A4)
   (layers
-    (0 F.Cu signal hide)
+    (0 F.Cu signal)
     (1 GND power hide)
     (2 VCC power hide)
@@
     (add_net USB-DPC)
   )
-  (module kicad-libraries:LED-RGB-LP (layer F.Cu)
-    (at 98.2 64.5 90)
-    (fp_text reference LED101 (at 0 0 90) (layer F.Fab)
+  (module kicad-libraries:WE-SL5 (layer F.Cu)
+    (at 150.5 135.65 180)
+    (fp_text reference T101 (at 0 0.5) (layer F.Fab)
       (effects (font (size 0.15 0.15) (thickness 0.0375)))
     )
-    (fp_text value EASV3015RGBA0 (at 0 -0.3 90) (layer F.Fab)
+    (fp_text value 744273222 (at 0 -0.5) (layer F.Fab)
       (effects (font (size 0.15 0.15) (thickness 0.0375)))
     )
-    (fp_line (start -1 -1.4) (end 1 -1.4) (layer F.Fab) (width 0.1))
-    (fp_line (start 1 -1.4) (end 1 -8.4) (layer F.Fab) (width 0.1))
-    (fp_line (start 1 -8.4) (end -1 -8.4) (layer F.Fab) (width 0.1))
-    (fp_line (start -1 -8.4) (end -1 -1.4) (layer F.Fab) (width 0.1))
-    (fp_line (start -1.5 -0.5) (end -1.5 0.2) (layer F.Fab) (width 0.025))
-    (fp_line (start 1.5 -0.5) (end -1.5 -0.5) (layer F.Fab) (width 0.025))
-    (fp_line (start 1.5 0.2) (end 1.5 -0.5) (layer F.Fab) (width 0.025))
-    (fp_line (start -1.5 0.2) (end 1.5 0.2) (layer F.Fab) (width 0.025))
-    (fp_arc (start 0 -0.5) (end -0.8 -0.5) (angle 90) (layer F.Fab) (width 0.025))
-    (fp_arc (start 0 -0.5) (end 0 -1.3) (angle 90) (layer F.Fab) (width 0.025))
-    (pad 3 smd rect (at -0.425 0.22 90) (size 0.55 0.34) (layers F.Cu F.Paste F.Mask)
-      (net 49 "Net-(LED101-Pad3)"))
-    (pad 2 smd rect (at 0.425 0.22 90) (size 0.55 0.34) (layers F.Cu F.Paste F.Mask)
-      (net 48 "Net-(LED101-Pad2)"))
-    (pad 4 smd rect (at -1.425 0 90) (size 0.55 0.78) (layers F.Cu F.Paste F.Mask)
-      (net 47 "Net-(LED101-Pad4)"))
-    (pad 1 smd rect (at 1.425 0 90) (size 0.55 0.78) (layers F.Cu F.Paste F.Mask)
-      (net 2 3V3))
-    (pad "" np_thru_hole circle (at 0 -2.4 90) (size 1.5 1.5) (drill 1.5) (layers *.Cu *.Mask))
+    (fp_line (start -5 4.4) (end -5 -4.4) (layer F.Fab) (width 0.1))
+    (fp_line (start 5 4.4) (end -5 4.4) (layer F.Fab) (width 0.1))
+    (fp_line (start 5 -4.4) (end 5 4.4) (layer F.Fab) (width 0.1))
+    (fp_line (start -5 -4.4) (end 5 -4.4) (layer F.Fab) (width 0.1))
+    (fp_circle (center -3.5 -2) (end -3.2 -1.7) (layer F.Fab) (width 0.1))
+    (pad 2 smd rect (at -3.81 3.11 180) (size 2.7 2.7) (layers F.Cu F.Paste F.Mask)
+      (net 93 AGNDA))
+    (pad 3 smd rect (at 3.81 3.11 180) (size 2.7 2.7) (layers F.Cu F.Paste F.Mask)
+      (net 104 "Net-(C120-Pad2)"))
+    (pad 4 smd rect (at 3.81 -3.11 180) (size 2.7 2.7) (layers F.Cu F.Paste F.Mask)
+      (net 85 "Net-(C119-Pad2)"))
+    (pad 1 smd rect (at -3.81 -3.11 180) (size 2.7 2.7) (layers F.Cu F.Paste F.Mask)
+      (net 96 "Net-(C121-Pad1)"))
+    (model ${KICAD_SYMBOL_DIR}/3d/Inductors/WE-SL5.wrl
+      (at (xyz 0 0 0))
+      (scale (xyz 1 1 1))
+      (rotate (xyz 0 0 0))
+    )
   )
   (module kicad-libraries:Fiducial_Mark (layer B.Cu)
@@
     )
   )
-  (module kicad-libraries:WE-SL5 (layer F.Cu)
-    (at 150.5 135.65)
-    (fp_text reference T101 (at 0 0.5) (layer F.Fab)
-      (effects (font (size 0.15 0.15) (thickness 0.0375)))
-    )
-    (fp_text value 744273222 (at 0 -0.5) (layer F.Fab)
-      (effects (font (size 0.15 0.15) (thickness 0.0375)))
-    )
-    (fp_line (start -5 4.4) (end -5 -4.4) (layer F.Fab) (width 0.1))
-    (fp_line (start 5 4.4) (end -5 4.4) (layer F.Fab) (width 0.1))
-    (fp_line (start 5 -4.4) (end 5 4.4) (layer F.Fab) (width 0.1))
-    (fp_line (start -5 -4.4) (end 5 -4.4) (layer F.Fab) (width 0.1))
-    (fp_circle (center -3.5 1.5) (end -3.2 1.8) (layer F.Fab) (width 0.1))
-    (pad 4 smd rect (at -3.81 3.11) (size 2.7 2.7) (layers F.Cu F.Paste F.Mask)
-      (net 85 "Net-(C119-Pad2)"))
-    (pad 3 smd rect (at 3.81 3.11) (size 2.7 2.7) (layers F.Cu F.Paste F.Mask)
-      (net 96 "Net-(C121-Pad1)"))
-    (pad 2 smd rect (at 3.81 -3.11) (size 2.7 2.7) (layers F.Cu F.Paste F.Mask)
-      (net 93 AGNDA))
-    (pad 1 smd rect (at -3.81 -3.11) (size 2.7 2.7) (layers F.Cu F.Paste F.Mask)
-      (net 104 "Net-(C120-Pad2)"))
-    (model Inductors/WE-SL5.wrl
-      (at (xyz 0 0 0))
-      (scale (xyz 1 1 1))
-      (rotate (xyz 0 0 0))
-    )
-  )
   (module C0402F (layer F.Cu)
     (at 156.85 98 90)
@@
     )
   )
+  (module LED-RGB-LP (layer F.Cu)
+    (at 98.2 64.5 90)
+    (fp_text reference LED101 (at 0 0 90) (layer F.Fab)
+      (effects (font (size 0.15 0.15) (thickness 0.0375)))
+    )
+    (fp_text value EASV3015RGBA0 (at 0 -0.3 90) (layer F.Fab)
+      (effects (font (size 0.15 0.15) (thickness 0.0375)))
+    )
+    (fp_arc (start 0 -0.5) (end 0 -1.3) (angle 90) (layer F.Fab) (width 0.025))
+    (fp_arc (start 0 -0.5) (end -0.8 -0.5) (angle 90) (layer F.Fab) (width 0.025))
+    (fp_line (start -1.5 0.2) (end 1.5 0.2) (layer F.Fab) (width 0.025))
+    (fp_line (start 1.5 0.2) (end 1.5 -0.5) (layer F.Fab) (width 0.025))
+    (fp_line (start 1.5 -0.5) (end -1.5 -0.5) (layer F.Fab) (width 0.025))
+    (fp_line (start -1.5 -0.5) (end -1.5 0.2) (layer F.Fab) (width 0.025))
+    (fp_line (start -1 -8.4) (end -1 -1.4) (layer F.Fab) (width 0.1))
+    (fp_line (start 1 -8.4) (end -1 -8.4) (layer F.Fab) (width 0.1))
+    (fp_line (start 1 -1.4) (end 1 -8.4) (layer F.Fab) (width 0.1))
+    (fp_line (start -1 -1.4) (end 1 -1.4) (layer F.Fab) (width 0.1))
+    (pad "" np_thru_hole circle (at 0 -2.4 90) (size 1.5 1.5) (drill 1.5) (layers *.Cu *.Mask))
+    (pad 1 smd rect (at 1.425 0 90) (size 0.55 0.78) (layers F.Cu F.Paste F.Mask)
+      (net 2 3V3))
+    (pad 4 smd rect (at -1.425 0 90) (size 0.55 0.78) (layers F.Cu F.Paste F.Mask)
+      (net 47 "Net-(LED101-Pad4)"))
+    (pad 2 smd rect (at 0.425 0.22 90) (size 0.55 0.34) (layers F.Cu F.Paste F.Mask)
+      (net 48 "Net-(LED101-Pad2)"))
+    (pad 3 smd rect (at -0.425 0.22 90) (size 0.55 0.34) (layers F.Cu F.Paste F.Mask)
+      (net 49 "Net-(LED101-Pad3)"))
+  )
   (gr_text tinkerforge.com (at 180.8 144.5) (layer B.SilkS)

Commit message: drc
Routing:
- net VCCPWRA: track 57.1 -> 53.6 mm, vias 13 -> 12
Changed lines of the file:
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@@
     (thickness 1.6)
     (drawings 29)
-    (tracks 1555)
+    (tracks 1551)
     (zones 0)
     (modules 131)
@@
     (1 GND power hide)
     (2 VCC power hide)
-    (31 B.Cu signal hide)
+    (31 B.Cu signal)
     (32 B.Adhes user)
-    (33 F.Adhes user)
+    (33 F.Adhes user hide)
     (34 B.Paste user)
     (35 F.Paste user)
@@
     (pad 3 smd rect (at -0.425 0.22 90) (size 0.55 0.34) (layers F.Cu F.Paste F.Mask)
       (net 49 "Net-(LED101-Pad3)"))
+    (model LED_SMD/LED_RGB_LP.wrl
+      (at (xyz 0 0 0))
+      (scale (xyz 1 1 1))
+      (rotate (xyz 0 0 0))
+    )
   )
   (gr_text tinkerforge.com (at 180.8 144.5) (layer B.SilkS)
@@
   (segment (start 170.15 124.1) (end 170.15 124.55) (width 0.4) (layer B.Cu) (net 94))
   (segment (start 170.15 124.55) (end 169.65 125.05) (width 0.4) (layer B.Cu) (net 94))
-  (via (at 172 124.1) (size 0.55) (drill 0.25) (layers F.Cu B.Cu) (net 94))
-  (segment (start 172.75 124.1) (end 172 124.1) (width 0.3) (layer B.Cu) (net 94))
-  (segment (start 172 124.1) (end 170.6 124.1) (width 0.3) (layer F.Cu) (net 94))
-  (segment (start 170.6 124.1) (end 169.65 125.05) (width 0.3) (layer F.Cu) (net 94))
   (via (at 170.85 120.5) (size 0.55) (drill 0.25) (layers F.Cu B.Cu) (net 94))
   (segment (start 171.7 120.3) (end 171.05 120.3) (width 0.3) (layer B.Cu) (net 94))
