File: hardware/di8.kicad_pcb (KiCad board)
At the start: 4 copper layers, 100 x 85 mm, 131 parts, among them J101 TNG-Power-TOP, J102 TNG-Power-BTM, J103 TNG-Data-TOP, J104 TNG-Data-BTM, P102 Debug, P103 PE, P201 INPUT0, P202 INPUT1, P203 INPUT2, P204 INPUT3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

Commit message: fix values
Parts:
- C127, C128: value 4.7nF/2kV -> 1nF/2kV
- R101: value 510 -> 1k

Commit message: fix value
Parts:
- C115: value TBD -> 2.2uF

Commit message: add version 1.2
fix footprints
Parts:
- C108, C109: value TBD -> 33pF
- C111: value TBD -> 100µF; footprint kicad-libraries:ELKO_83 -> kicad-libraries:ELKO_63
- C122, C123, C124: footprint kicad-libraries:ELKO_83 -> kicad-libraries:ELKO_63
- D201, D202, D211, D212, D213, D214, D215, D216: footprint SOD-123 -> kicad-libraries:SOD-123FL
- R109: footprint kicad-libraries:R0603F -> kicad-libraries:R0402F
- X101: value TBD -> 8MHz
- moved C124 1.05 mm to (160.8, 117.7)
- moved C122 1.05 mm to (169.7, 117.7)
- moved C111 0.80 mm to (165.4, 90.2)
- moved C123 0.60 mm to (161.5, 134.5)
- moved R109 0.60 mm to (175.3, 105.7)
- moved D201 0.40 mm to (102.9, 85.9), turned to 270 degrees
- moved D202 0.40 mm to (102.9, 93.1), turned to 90 degrees
- moved D211 0.40 mm to (102.9, 101.9), turned to 270 degrees
- moved D212 0.40 mm to (102.9, 117.9), turned to 270 degrees
- moved D213 0.40 mm to (102.9, 133.9), turned to 270 degrees
- moved D214 0.40 mm to (102.9, 109.1), turned to 90 degrees
- moved D215 0.40 mm to (102.9, 125.1), turned to 90 degrees
- moved D216 0.40 mm to (102.9, 141.1), turned to 90 degrees
- moved R201 0.40 mm to (99.7, 91.2)
- moved R202 0.40 mm to (99.7, 87.8)
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Connections:
- J101 pad 21: (no net) -> Net-(J101-Pad21)
- J101 pad 22: (no net) -> Net-(J101-Pad22)
- J101 pad 23: (no net) -> Net-(J101-Pad23)
- J101 pad 24: (no net) -> Net-(J101-Pad24)
- J101 pad 25: (no net) -> Net-(J101-Pad25)
- J101 pad 26: (no net) -> Net-(J101-Pad26)
- J101 pad 27: (no net) -> Net-(J101-Pad27)
- J101 pad 28: (no net) -> Net-(J101-Pad28)
- J101 pad 29: (no net) -> Net-(J101-Pad29)
- J101 pad 30: (no net) -> Net-(J101-Pad30)
- J102 pad 21: (no net) -> Net-(J102-Pad21)
- J102 pad 22: (no net) -> Net-(J102-Pad22)
- J102 pad 23: (no net) -> Net-(J102-Pad23)
- J102 pad 24: (no net) -> Net-(J102-Pad24)
- J102 pad 25: (no net) -> Net-(J102-Pad25)
- J102 pad 26: (no net) -> Net-(J102-Pad26)
- J102 pad 27: (no net) -> Net-(J102-Pad27)
- J102 pad 28: (no net) -> Net-(J102-Pad28)
- J102 pad 29: (no net) -> Net-(J102-Pad29)
- J102 pad 30: (no net) -> Net-(J102-Pad30)
- J103 pad 35: (no net) -> Net-(J103-Pad35)
- J103 pad 37: (no net) -> Net-(J103-Pad37)
- U101 pad 11: (no net) -> Net-(U101-Pad11)
- U101 pad 17: (no net) -> Net-(U101-Pad17)
- U101 pad 2: (no net) -> Net-(U101-Pad2)
- U101 pad 21: (no net) -> Net-(U101-Pad21)
- U101 pad 22: (no net) -> Net-(U101-Pad22)
- U101 pad 26: (no net) -> Net-(U101-Pad26)
- U101 pad 27: (no net) -> Net-(U101-Pad27)
- U101 pad 28: (no net) -> Net-(U101-Pad28)
- U101 pad 3: (no net) -> Net-(U101-Pad3)
- U101 pad 4: (no net) -> Net-(U101-Pad4)
- U101 pad 46: (no net) -> Net-(U101-Pad46)
- U101 pad 7: (no net) -> Net-(U101-Pad7)
- U104 pad 7: (no net) -> Net-(U104-Pad7)
- U104 pad 8: (no net) -> Net-(U104-Pad8)
- U106 pad 12: (no net) -> Net-(U106-Pad12)
- U106 pad 2: (no net) -> Net-(U106-Pad2)
- U201 pad 12: (no net) -> Net-(U201-Pad12)
- U201 pad 13: (no net) -> Net-(U201-Pad13)
- U201 pad 6: (no net) -> Net-(U201-Pad6)
- U201 pad 7: (no net) -> Net-(U201-Pad7)
- U202 pad 12: (no net) -> Net-(U202-Pad12)
- U202 pad 13: (no net) -> Net-(U202-Pad13)
- U202 pad 6: (no net) -> Net-(U202-Pad6)
- U202 pad 7: (no net) -> Net-(U202-Pad7)
- U203 pad 12: (no net) -> Net-(U203-Pad12)
- U203 pad 13: (no net) -> Net-(U203-Pad13)
- U203 pad 6: (no net) -> Net-(U203-Pad6)
- U203 pad 7: (no net) -> Net-(U203-Pad7)
- U204 pad 12: (no net) -> Net-(U204-Pad12)
- U204 pad 13: (no net) -> Net-(U204-Pad13)
- U204 pad 6: (no net) -> Net-(U204-Pad6)
- U204 pad 7: (no net) -> Net-(U204-Pad7)
Routing:
- net AGND: track 123.3 -> 127.2 mm
- added copper zone on F.Cu, net AGNDA
Other:
- board text added: "Copyright Tinkerforge GmbH 2020. This documentation describes Open Hardware and is licensed under the CERN OHL v. 1.1. You may redistribute and modify this documentation under the terms of the CERN OHL v.1.1. (http://ohwr.org/cernohl). This documentation is distributed WITHOUT ANY EXPRESS OR IMPLIED WARRANTY, INCLUDING OF MERCHANTABILITY, SATISFACTORY QUALITY AND FITNESS FOR A PARTICULAR PURPOSE.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"
- board text added: "DI 8P REV 1.2"
- board text removed: "DI 8P REV 1.1"

Commit message: specify capactors
Parts:
- C113, C114: value TBD/47pF -> 47pF

Commit message: fix stuff
Parts:
- C110, C202, C203, C205, C206, C207, C208, C209, C210: footprint C0805 -> kicad-libraries:C0805E

Commit message: fix values
Parts:
- C111: value 100µF -> 100uF
- C118: value 10µF/50V -> 10uF/50V
- C121, C125, C126: value 10µF/35V -> 10uF/35V
- C122, C123, C124: value 100µF/35V -> 100uF/35V
Changed lines of the file:
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@@
       (effects (font (size 0.3 0.3) (thickness 0.075)))
     )
-    (fp_text value 10µF/50V (at 0 -0.65 -180) (layer F.Fab)
+    (fp_text value 10uF/50V (at 0 -0.65 -180) (layer F.Fab)
       (effects (font (size 0.3 0.3) (thickness 0.075)))
     )
@@
       (effects (font (size 0.3 0.3) (thickness 0.075)) (justify mirror))
     )
-    (fp_text value 10µF/35V (at 0 0.65 90) (layer B.Fab)
+    (fp_text value 10uF/35V (at 0 0.65 90) (layer B.Fab)
       (effects (font (size 0.3 0.3) (thickness 0.075)) (justify mirror))
     )
@@
       (effects (font (size 0.3 0.3) (thickness 0.075)))
     )
-    (fp_text value 10µF/35V (at 0 -0.65) (layer F.Fab)
+    (fp_text value 10uF/35V (at 0 -0.65) (layer F.Fab)
       (effects (font (size 0.3 0.3) (thickness 0.075)))
     )
@@
       (effects (font (size 0.3 0.3) (thickness 0.075)))
     )
-    (fp_text value 10µF/35V (at 0 -0.65) (layer F.Fab)
+    (fp_text value 10uF/35V (at 0 -0.65) (layer F.Fab)
       (effects (font (size 0.3 0.3) (thickness 0.075)))
     )
@@
       (effects (font (size 0.59944 0.59944) (thickness 0.12446)))
     )
-    (fp_text value 100µF (at 0.95 -0.375) (layer F.Fab)
+    (fp_text value 100uF (at 0.95 -0.375) (layer F.Fab)
       (effects (font (size 0.59944 0.59944) (thickness 0.12446)))
     )
@@
       (effects (font (size 0.59944 0.59944) (thickness 0.12446)))
     )
-    (fp_text value 100µF/35V (at 0.95 -0.375 90) (layer F.Fab)
+    (fp_text value 100uF/35V (at 0.95 -0.375 90) (layer F.Fab)
       (effects (font (size 0.59944 0.59944) (thickness 0.12446)))
     )
@@
       (effects (font (size 0.59944 0.59944) (thickness 0.12446)))
     )
-    (fp_text value 100µF/35V (at 0.95 -0.375) (layer F.Fab)
+    (fp_text value 100uF/35V (at 0.95 -0.375) (layer F.Fab)
       (effects (font (size 0.59944 0.59944) (thickness 0.12446)))
     )
@@
       (effects (font (size 0.59944 0.59944) (thickness 0.12446)))
     )
-    (fp_text value 100µF/35V (at 0.95 -0.375 90) (layer F.Fab)
+    (fp_text value 100uF/35V (at 0.95 -0.375 90) (layer F.Fab)
       (effects (font (size 0.59944 0.59944) (thickness 0.12446)))
     )

Commit message: all footprints updated
Parts:
- C101, C102, C103, C104, C105, C106, C107, C108, C109, C112, C113, C114, C116, C117, C204, C211, C212, C213: footprint C0402F -> kicad-libraries:C0402F
- C115: footprint C0603F -> kicad-libraries:C0603F
- C118, C119, C120, C121, C125, C126, C127, C128: footprint C1206 -> kicad-libraries:C1206
- D203, D204, D205, D206, D207, D208, D209, D210: footprint LED-LP -> kicad-libraries:LED-LP
- J101, J103: footprint TNG-40-TOP -> kicad-libraries:TNG-40-TOP
- J102, J104: footprint TNG-40-BTM -> kicad-libraries:TNG-40-BTM
- L101, L102, L103, L104, R203, R204, R211, R212, R213, R214, R215, R216: footprint R0603F -> kicad-libraries:R0603F
- L105: footprint WE-CNSW-0603 -> kicad-libraries:WE-CNSW-0603
- LED101: footprint LED-RGB-LP -> kicad-libraries:LED-RGB-LP
- P201, P202, P203, P204: footprint OQ_4P -> kicad-libraries:OQ_4P
- R101, R102, R103, R104, R105, R106, R107, R108: footprint R0402F -> kicad-libraries:R0402F
- R201, R202, R205, R206, R207, R208, R209, R210: footprint RMELF -> kicad-libraries:RMELF
- U103: footprint SOT563-SPEC -> kicad-libraries:SOT563-SPEC
- U201, U202, U203, U204: footprint SSOP16 -> kicad-libraries:SSOP16

Commit message: default is non implemented
Parts:
- C101, C102, C103, C104, C105, C106, C107, C108, C109, C112, C113, C114, C116, C117, C204, C211, C212, C213: footprint kicad-libraries:C0402F -> C0402F
- C115: footprint kicad-libraries:C0603F -> C0603F
- C118, C121, C125, C126, C127, C128: footprint kicad-libraries:C1206 -> C1206
- C119, C120: value 1nF 2kV -> 0; footprint kicad-libraries:C1206 -> C1206
- D203, D204, D205, D206, D207, D208, D209, D210: footprint kicad-libraries:LED-LP -> LED-LP
- J101, J103: footprint kicad-libraries:TNG-40-TOP -> TNG-40-TOP
- J102, J104: footprint kicad-libraries:TNG-40-BTM -> TNG-40-BTM
- L101, L102, L103, L104, R203, R204, R211, R212, R213, R214, R215, R216: footprint kicad-libraries:R0603F -> R0603F
- L105: footprint kicad-libraries:WE-CNSW-0603 -> WE-CNSW-0603
- LED101: footprint kicad-libraries:LED-RGB-LP -> LED-RGB-LP
- P201, P202, P203, P204: footprint kicad-libraries:OQ_4P -> OQ_4P
- R101, R102, R103, R104, R105, R106, R107, R108: footprint kicad-libraries:R0402F -> R0402F
- R201, R202, R205, R206, R207, R208, R209, R210: footprint kicad-libraries:RMELF -> RMELF
- U103: footprint kicad-libraries:SOT563-SPEC -> SOT563-SPEC
- U104: value TEL10 -> DNP
- U201, U202, U203, U204: footprint kicad-libraries:SSOP16 -> SSOP16
